File: OpAmpDevBoardProject/OpAmpDevBoardProject.kicad_pcb (KiCad board)
At the start: 2 copper layers, 105 parts, among them J101 Conn_01x07, J102 Conn_01x01_Pin, J103 Conn_01x01_Pin, J104 Conn_01x01_Pin, J105 Conn_01x01_Pin, J106 Conn_01x01_Pin, J107 Conn_01x01_Pin, J108 Conn_01x01_Pin, J109 Conn_01x07_Socket, J110 227161-2, J111 227161-2, J112 Conn_01x01_Pin, J113 Conn_01x01_Pin, J114 Conn_01x01_Pin, J115 Conn_01x01_Pin, J116 227161-2, J117 Conn_01x01_Pin, J118 Conn_01x01_Pin, J119 Conn_01x01_Pin, J120 Conn_01x01_Pin, J121 227161-2, J122 Conn_01x01_Pin, J123 Conn_01x01_Pin, J124 Conn_01x01_Pin, J125 Conn_01x01_Pin, J126 Conn_01x01_Pin, J127 Conn_01x01_Pin, J128 Conn_01x01_Pin, SW101 SW_SPST, SW102 SW_SPST, SW103 SW_SPST, SW104 SW_SPST, SW105 SW_SPST, SW106 SW_SPST, SW107 SW_SPST, SW108 SW_SPST, SW109 SW_SPST, SW110 SW_SPST, SW111 SW_SPST, SW112 SW_SPST, SW113 SW_SPST, SW114 SW_SPST, SW115 SW_SPST, SW116 SW_SPST, SW117 SW_SPST, SW118 SW_SPST, SW119 SW_SPST, SW120 SW_SPST, SW121 SW_SPST, SW122 SW_SPST, SW123 SW_SPST, SW124 SW_SPST, SW125 SW_SPST, SW126 SW_SPST, SW127 SW_SPST, SW128 SW_SPST, SW129 SW_SPST, SW130 SW_SPST, SW131 SW_SPST, SW132 SW_SPST, SW133 SW_SPST, SW134 SW_SPST, SW135 SW_SPST, SW136 SW_SPST, SW137 SW_SPST, SW138 SW_SPST, SW139 SW_SPST, SW140 SW_SPST, SW141 SW_SPST, SW142 SW_SPST, SW143 SW_SPST, SW144 SW_SPST, SW145 SW_SPST, SW146 SW_SPST, U101 DoualOutOpAmpGeneric

Commit message: added double switch and started changing schematic
Parts:
- added SW147: SW_SPST, OpAmpDevBoard_Mouser:SS12SDP2, F.Cu at (216.0, 202.0)
- added SW148: SW_SPST, OpAmpDevBoard_Mouser:SS12SDP2, F.Cu at (216.0, 102.0)
- H101, H102, H103, H104: moved to B.Cu
- moved RV101 340.5 mm to (249.5, 188.1), turned to 90 degrees
- moved H101 338.9 mm to (54.0, 245.0), turned to 180 degrees
- moved SW104 309.1 mm to (224.0, 241.0), turned to 180 degrees
- moved SW102 299.9 mm to (243.9, 216.0), turned to 90 degrees
- moved SW106 299.0 mm to (243.9, 228.0), turned to 90 degrees
- moved RV102 296.5 mm to (249.5, 128.1), turned to 90 degrees
- moved SW103 286.9 mm to (244.0, 205.0), turned to 90 degrees
- moved SW101 284.2 mm to (244.0, 194.0), turned to 90 degrees
- moved J101 283.1 mm to (47.0, 143.4)
- moved J109 268.8 mm to (61.0, 143.4)
- moved C101 268.1 mm to (246.0, 234.0), turned to 180 degrees
- moved J102 261.9 mm to (224.0, 228.0)
- moved C107 260.2 mm to (197.0, 237.0), turned to -90 degrees
- moved H103 255.5 mm to (54.0, 55.0), turned to 180 degrees
- moved C106 250.0 mm to (182.0, 219.0), turned to 90 degrees
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Connections:
- C102 pad 2: Net-(J103-Pin_1) -> Net-(J127-Pin_1)
- C105 pad 2: Net-(J102-Pin_1) -> Net-(J107-Pin_1)
- J107 pad 1: Net-(J102-Pin_1) -> Net-(J107-Pin_1)
- J127 pad 1: Net-(J103-Pin_1) -> Net-(J127-Pin_1)
- SW107 pad 1: Net-(J103-Pin_1) -> Net-(J127-Pin_1)
- SW108 pad 1: Net-(J103-Pin_1) -> Net-(J127-Pin_1)
- SW109 pad 2: Net-(J103-Pin_1) -> Net-(J127-Pin_1)
- SW110 pad 2: Net-(J103-Pin_1) -> Net-(J127-Pin_1)
- SW115 pad 2: Net-(J103-Pin_1) -> Net-(J127-Pin_1)
- SW116 pad 2: Net-(J103-Pin_1) -> Net-(J127-Pin_1)
- SW121 pad 2: Net-(J102-Pin_1) -> Net-(J107-Pin_1)
- SW122 pad 2: Net-(J102-Pin_1) -> Net-(J107-Pin_1)
- SW123 pad 1: Net-(J102-Pin_1) -> Net-(J107-Pin_1)
- SW124 pad 1: Net-(J102-Pin_1) -> Net-(J107-Pin_1)
- SW125 pad 2: Net-(J102-Pin_1) -> Net-(J107-Pin_1)
- SW126 pad 2: Net-(J102-Pin_1) -> Net-(J107-Pin_1)
- SW135 pad 2: Net-(J102-Pin_1) -> Net-(J107-Pin_1)
- SW138 pad 2: Net-(J103-Pin_1) -> Net-(J127-Pin_1)
Other:
- board outline added: 257 x 210 mm
- copper layers 2 -> 4

Commit message: late night fu me
Parts:
- removed SW143: SW_SPST, OpAmpDevBoard_Mouser:SS12SDP2
- added JP101: Jumper_2_Small_Bridged, Connector_PinHeader_2.54mm:PinHeader_1x02_P2.54mm_Vertical, F.Cu at (89.5, 169.0)
- added JP102: Jumper_2_Small_Bridged, Connector_PinHeader_2.54mm:PinHeader_1x02_P2.54mm_Vertical, F.Cu at (121.5, 169.0)
- added JP103: Jumper_2_Small_Bridged, Connector_PinHeader_2.54mm:PinHeader_1x02_P2.54mm_Vertical, F.Cu at (248.0, 172.0)
- added JP104: Jumper_2_Small_Bridged, Connector_PinHeader_2.54mm:PinHeader_1x02_P2.54mm_Vertical, F.Cu at (88.5, 135.0)
- added JP105: Jumper_2_Small_Bridged, Connector_PinHeader_2.54mm:PinHeader_1x02_P2.54mm_Vertical, F.Cu at (121.5, 135.0)
- added JP106: Jumper_2_Small_Bridged, Connector_PinHeader_2.54mm:PinHeader_1x02_P2.54mm_Vertical, F.Cu at (247.5, 132.0)
- added SW149: SS22S, OpAmpDevBoard_Mouser:SS22SDP2, F.Cu at (93.0, 193.0)
- SW101, SW131, SW139, SW140, SW142: value SW_SPST -> SS22S; footprint OpAmpDevBoard_Mouser:SS12SDP2 -> OpAmpDevBoard_Mouser:SS22SDP2
- moved SW140 83.6 mm to (93.0, 114.0)
- moved SW139 33.5 mm to (126.1, 193.0)
- moved SW142 32.9 mm to (126.0, 114.0)
- moved SW131 1.54 mm to (244.0, 108.5)
- moved SW101 1.00 mm to (244.0, 193.0)
- moved J112 0.38 mm to (64.0, 80.5)
- moved SW134 0.08 mm to (125.5, 202.0)
Connections:
- RV101 pad 2: Net-(J102-Pin_1) -> Net-(RV101-Pad2)
- RV101 pad 3: GND -> Net-(JP103-B)
- RV102 pad 2: Net-(J103-Pin_1) -> Net-(RV102-Pad2)
- RV102 pad 3: GND -> Net-(JP106-B)
- RV103 pad 1: Net-(SW139-B) -> Net-(RV103-Pad1)
- RV103 pad 2: Net-(J105-Pin_1) -> Net-(RV103-Pad2)
- RV103 pad 3: GND -> Net-(JP101-A)
- RV104 pad 1: Net-(SW140-B) -> Net-(RV104-Pad1)
- RV104 pad 2: Net-(J106-Pin_1) -> Net-(RV104-Pad2)
- RV104 pad 3: GND -> Net-(JP102-A)
- RV106 pad 1: Net-(SW142-B) -> Net-(RV106-Pad1)
- RV106 pad 2: Net-(J125-Pin_1) -> Net-(RV106-Pad2)
- RV106 pad 3: GND -> Net-(JP104-A)
- RV107 pad 1: Net-(SW143-B) -> Net-(RV107-Pad1)
- RV107 pad 2: Net-(J126-Pin_1) -> Net-(RV107-Pad2)
- RV107 pad 3: GND -> Net-(JP105-A)
- SW139 pad 1: Net-(J104-Pin_1) -> Net-(J105-Pin_1)
- SW139 pad 2: Net-(SW139-B) -> Net-(RV104-Pad1)
- SW140 pad 1: Net-(J105-Pin_1) -> Net-(J110-Signal)
- SW140 pad 2: Net-(SW140-B) -> Net-(RV106-Pad1)
- SW142 pad 1: Net-(J110-Signal) -> Net-(J125-Pin_1)
- SW142 pad 2: Net-(SW142-B) -> Net-(RV107-Pad1)
Routing:
- net Net-(J103-Pin_1): track 0.00 -> 266.5 mm, vias 0 -> 3
- net Net-(J102-Pin_1): track 0.00 -> 256.0 mm, vias 0 -> 3
- net /V-: track 0.00 -> 246.7 mm
- net /Div2: track 0.00 -> 245.5 mm
- net /Sleep: track 0.00 -> 244.8 mm, vias 0 -> 1
- net /Div1: track 0.00 -> 242.5 mm
- net /Act: track 0.00 -> 241.7 mm, vias 0 -> 1
- net /V+: track 0.00 -> 235.9 mm
- net Net-(J119-Pin_1): track 0.00 -> 201.2 mm, vias 0 -> 3
- net Net-(J107-Pin_1): track 0.00 -> 163.1 mm, vias 0 -> 3
- net Net-(J127-Pin_1): track 0.00 -> 162.2 mm
- net Net-(J116-Signal): track 0.00 -> 155.3 mm, vias 0 -> 3
- net Net-(J125-Pin_1): track 0.00 -> 144.4 mm, vias 0 -> 5
- net Net-(J105-Pin_1): track 0.00 -> 143.6 mm, vias 0 -> 4
- net Net-(J106-Pin_1): track 0.00 -> 128.5 mm, vias 0 -> 5
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- added copper zone on B.Cu, net GND
- added copper zone on F.Cu, net GND
- added copper zone on In1.Cu, net GND
- added copper zone on In2.Cu, net GND
Other:
- board text added: "ACT"
- board text added: "Act"
- board text added: "DIV 1"
- board text added: "DIV 2"
- board text added: "Div 1"
- board text added: "Div 2"
- board text added: "Fabian Glutz https://github.com/Gehtschon/OpAmpDevBoard"
- board text added: "GND"
- board text added: "JLCJLCJLCJLC"
- board text added: "OUT1"
- board text added: "OUT2"
- board text added: "OpAmp DevBoard V.0.1"
- board text added: "Open → Variable Resistor Closed → Voltage Divider"
- board text added: "SIG+"
- board text added: "SIG-"
- board text added: "Sig+"
- board text added: "Sig-"
- board text added: "Sleep"
- board text added: "Switch towards symbol = Activate"
- board text added: "V+"
- board text added: "V-"

Commit message: added gnd connectors
Parts:
- added J129: Conn_01x01_Pin, Connector_PinHeader_2.54mm:PinHeader_1x01_P2.54mm_Vertical, F.Cu at (61.5, 55.0)
- added J130: Conn_01x01_Pin, Connector_PinHeader_2.54mm:PinHeader_1x01_P2.54mm_Vertical, F.Cu at (283.5, 55.5)
- added J131: Conn_01x01_Pin, Connector_PinHeader_2.54mm:PinHeader_1x01_P2.54mm_Vertical, F.Cu at (61.5, 245.0)
- added J132: Conn_01x01_Pin, Connector_PinHeader_2.54mm:PinHeader_1x01_P2.54mm_Vertical, F.Cu at (283.5, 245.0)
